Commit message: removed dependency on uos_tools macro

File: fanuc_lrmate200id_support/urdf/lrmate200id_macro.xacro (robot description, xacro)
@@ -5,5 +5,5 @@
   <xacro:include filename="$(find fanuc_lrmate200id_support)/urdf/lrmate200id.gazebo.xacro"/>
   <xacro:include filename="$(find fanuc_lrmate200id_support)/urdf/lrmate200id.transmission.xacro"/>
-  <xacro:include filename="$(find uos_common_urdf)/common.xacro"/>
+  <!--<xacro:include filename="$(find uos_common_urdf)/common.xacro"/>-->
   <xacro:macro name="fanuc_lrmate200id" params="prefix">
     <link name="${prefix}base_link">
@@ -21,5 +21,10 @@
         </geometry>
       </collision>
-      <xacro:box_inertial x="0.19" y=".19" z=".17" mass="4" />
+      <!--<xacro:box_inertial x="0.19" y=".19" z=".17" mass="4" />-->
+      <inertial>
+        <mass value="4"/>
+        <origin xyz="0 0 0"/>
+        <inertia ixx="0.021666658" ixy="0.0" ixz="0.0" iyy="0.021666658" iyz="0.0" izz="0.02406665704"/>
+      </inertial>
     </link>
     <link name="${prefix}link_1">
@@ -37,5 +42,10 @@
         </geometry>
       </collision>
-      <xacro:box_inertial x="0.14" y=".22" z=".22" mass="4" />
+      <!--<xacro:box_inertial x="0.14" y=".22" z=".22" mass="4" />-->
+      <inertial>
+        <mass value="4"/>
+        <origin xyz="0 0 0"/>
+        <inertia ixx="0.03226665376" ixy="0.0" ixz="0.0" iyy="0.0226666576" iyz="0.0" izz="0.0226666576"/>
+      </inertial>
     </link>
     <link name="${prefix}link_2">
@@ -53,5 +63,10 @@
         </geometry>
       </collision>
-      <xacro:box_inertial x="0.14" y=".20" z=".44" mass="5" />
+      <!--<xacro:box_inertial x="0.14" y=".20" z=".44" mass="5" />-->
+      <inertial>
+        <mass value="5"/>
+        <origin xyz="0 0 0"/>
+        <inertia ixx="0.0973332944" ixy="0.0" ixz="0.0" iyy="0.0888332978" iyz="0.0" izz="0.0248333234"/>
+      </inertial>
     </link>
     <link name="${prefix}link_3">
@@ -69,5 +84,10 @@
         </geometry>
       </collision>
-      <xacro:box_inertial x="0.14" y=".12" z=".13" mass="4" />
+      <!--<xacro:box_inertial x="0.14" y=".12" z=".13" mass="4" />-->
+      <inertial>
+        <mass value="4"/>
+        <origin xyz="0 0 0"/>
+        <inertia ixx="0.01043332916" ixy="0.0" ixz="0.0" iyy="0.0121666618" iyz="0.0" izz="0.0113333288"/>
+      </inertial>
     </link>
     <link name="${prefix}link_4">
@@ -85,5 +105,10 @@
         </geometry>
       </collision>
-      <xacro:box_inertial x="0.28" y=".10" z=".10" mass="5" />
+      <!--<xacro:box_inertial x="0.28" y=".10" z=".10" mass="5" />-->
+      <inertial>
+        <mass value="5"/>
+        <origin xyz="0 0 0"/>
+        <inertia ixx="0.00833333" ixy="0.0" ixz="0.0" iyy="0.0368333186" iyz="0.0" izz="0.0368333186"/>
+      </inertial>
     </link>
     <link name="${prefix}link_5">
@@ -101,5 +126,10 @@
         </geometry>
       </collision>
-      <xacro:box_inertial x="0.11" y=".09" z=".08" mass="1.5" />
+      <!--<xacro:box_inertial x="0.11" y=".09" z=".08" mass="1.5" />-->
+      <inertial>
+        <mass value="1.5"/>
+        <origin xyz="0 0 0"/>
+        <inertia ixx="0.001812499275" ixy="0.0" ixz="0.0" iyy="0.002312499075" iyz="0.0" izz="0.00252499899"/>
+      </inertial>
     </link>
     <link name="${prefix}link_6">
@@ -117,5 +147,10 @@
         </geometry>
       </collision>
-      <xacro:box_inertial x="0.01" y=".04" z=".04" mass=".25" />
+      <!--<xacro:box_inertial x="0.01" y=".04" z=".04" mass=".25" />-->
+      <inertial>
+        <mass value="0.25"/>
+        <origin xyz="0 0 0"/>
+        <inertia ixx="6.666664e-05" ixy="0.0" ixz="0.0" iyy="3.54166525e-05" iyz="0.0" izz="3.54166525e-05"/>
+      </inertial>
     </link>
     <link name="${prefix}tool0" />

Commit message: Added Gazebo controller support and ROS-I trajectory filters

File: fanuc_lrmate200id_support/urdf/lrmate200id_macro.xacro (robot description, xacro)
@@ -3,4 +3,6 @@
   <xacro:include filename="$(find fanuc_resources)/urdf/common_materials.xacro"/>
   <xacro:include filename="$(find fanuc_resources)/urdf/common_constants.xacro"/>
+  <xacro:include filename="$(find fanuc_lrmate200id_support)/urdf/lrmate200id.gazebo.xacro"/>
+  <xacro:include filename="$(find fanuc_lrmate200id_support)/urdf/lrmate200id.transmission.xacro"/>
   <xacro:macro name="fanuc_lrmate200id" params="prefix">
     <link name="${prefix}base_link">
@@ -18,4 +20,9 @@
         </geometry>
       </collision>
+      <inertial>
+        <mass value="4"/>
+        <origin xyz="0 0 0"/>
+        <inertia ixx="0.021666658" ixy="0.0" ixz="0.0" iyy="0.021666658" iyz="0.0" izz="0.02406665704"/>
+      </inertial>
     </link>
     <link name="${prefix}link_1">
@@ -33,4 +40,9 @@
         </geometry>
       </collision>
+      <inertial>
+        <mass value="4"/>
+        <origin xyz="0 0 0"/>
+        <inertia ixx="0.03226665376" ixy="0.0" ixz="0.0" iyy="0.0226666576" iyz="0.0" izz="0.0226666576"/>
+      </inertial>
     </link>
     <link name="${prefix}link_2">
@@ -48,4 +60,9 @@
         </geometry>
       </collision>
+      <inertial>
+        <mass value="5"/>
+        <origin xyz="0 0 0"/>
+        <inertia ixx="0.0973332944" ixy="0.0" ixz="0.0" iyy="0.0888332978" iyz="0.0" izz="0.0248333234"/>
+      </inertial>
     </link>
     <link name="${prefix}link_3">
@@ -63,4 +80,9 @@
         </geometry>
       </collision>
+      <inertial>
+        <mass value="4"/>
+        <origin xyz="0 0 0"/>
+        <inertia ixx="0.01043332916" ixy="0.0" ixz="0.0" iyy="0.0121666618" iyz="0.0" izz="0.0113333288"/>
+      </inertial>
     </link>
     <link name="${prefix}link_4">
@@ -78,4 +100,9 @@
         </geometry>
       </collision>
+      <inertial>
+        <mass value="5"/>
+        <origin xyz="0 0 0"/>
+        <inertia ixx="0.00833333" ixy="0.0" ixz="0.0" iyy="0.0368333186" iyz="0.0" izz="0.0368333186"/>
+      </inertial>
     </link>
     <link name="${prefix}link_5">
@@ -93,4 +120,9 @@
         </geometry>
       </collision>
+      <inertial>
+        <mass value="1.5"/>
+        <origin xyz="0 0 0"/>
+        <inertia ixx="0.001812499275" ixy="0.0" ixz="0.0" iyy="0.002312499075" iyz="0.0" izz="0.00252499899"/>
+      </inertial>
     </link>
     <link name="${prefix}link_6">
@@ -108,4 +140,9 @@
         </geometry>
       </collision>
+      <inertial>
+        <mass value="0.25"/>
+        <origin xyz="0 0 0"/>
+        <inertia ixx="6.666664e-05" ixy="0.0" ixz="0.0" iyy="3.54166525e-05" iyz="0.0" izz="3.54166525e-05"/>
+      </inertial>
     </link>
     <link name="${prefix}tool0" />
@@ -164,4 +201,6 @@
       <child link="${prefix}base"/>
     </joint>
+    <xacro:fanuc_transmission prefix="${prefix}"/>
+    <xacro:fanuc_gazebo prefix="${prefix}"/>
   </xacro:macro>
 </robot>
